File: STM32AppBoard.kicad_sch (KiCad schematic)
At the start: 23 parts, among them SW1 SW_Wuerth_450301014042, U1 DM-OLED096-636, U3 NUCLEO-L412KB, U4 JDY-08-jdy-08

Commit message: Update STM32AppBoard schematic and PCB layout
Parts:
- removed R1: LDR07, OptoDevice:R_LDR_5.1x4.3mm_P3.4mm_Vertical, symbol Sensor_Optical:LDR07
- removed SW1: SW_Wuerth_450301014042, Button_Switch_THT:SW_Slide-03_Wuerth-WS-SLTV_10x2.5x6.4_P2.54mm, symbol Switch:SW_Wuerth_450301014042
Other:
- moved on the sheet: D3, R10, R11, R9
Changed lines of the file:
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@@
 	)
 	(junction
-		(at 147.32 189.23)
+		(at 135.89 176.53)
 		(diameter 0)
 		(color 0 0 0 0)
@@
 	(wire
 		(pts
-			(xy 113.03 173.99) (xy 120.65 173.99)
+			(xy 101.6 161.29) (xy 109.22 161.29)
 		)
 		(stroke
@@
 	(wire
 		(pts
-			(xy 135.89 179.07) (xy 138.43 179.07)
+			(xy 124.46 166.37) (xy 127 166.37)
 		)
 		(stroke
@@
 	(wire
 		(pts
-			(xy 135.89 173.99) (xy 156.21 173.99)
+			(xy 124.46 161.29) (xy 144.78 161.29)
 		)
 		(stroke
@@
 	(wire
 		(pts
-			(xy 156.21 173.99) (xy 156.21 181.61)
+			(xy 144.78 161.29) (xy 144.78 168.91)
 		)
 		(stroke
@@
 	(wire
 		(pts
-			(xy 147.32 189.23) (xy 156.21 189.23)
+			(xy 135.89 176.53) (xy 144.78 176.53)
 		)
 		(stroke
@@
 	(wire
 		(pts
-			(xy 138.43 189.23) (xy 147.32 189.23)
+			(xy 127 176.53) (xy 135.89 176.53)
 		)
 		(stroke
@@
 	(wire
 		(pts
-			(xy 147.32 176.53) (xy 147.32 181.61)
+			(xy 135.89 163.83) (xy 135.89 168.91)
 		)
 		(stroke
@@
 	(wire
 		(pts
-			(xy 135.89 176.53) (xy 147.32 176.53)
+			(xy 124.46 163.83) (xy 135.89 163.83)
 		)
 		(stroke
@@
 	(wire
 		(pts
-			(xy 138.43 179.07) (xy 138.43 181.61)
+			(xy 127 166.37) (xy 127 168.91)
 		)
 		(stroke
@@
 	(wire
 		(pts
-			(xy 113.03 179.07) (xy 120.65 179.07)
+			(xy 101.6 166.37) (xy 109.22 166.37)
 		)
 		(stroke
@@
 	(wire
 		(pts
-			(xy 113.03 176.53) (xy 120.65 176.53)
+			(xy 101.6 163.83) (xy 109.22 163.83)
 		)
 		(stroke
@@
 	)
 	(label "PWM_B"
-		(at 113.03 179.07 0)
+		(at 101.6 166.37 0)
 		(effects
 			(font
@@
 	)
 	(label "PWM_R"
-		(at 113.03 173.99 0)
+		(at 101.6 161.29 0)
 		(effects
 			(font
@@
 	)
 	(label "PWM_G"
-		(at 113.03 176.53 0)
+		(at 101.6 163.83 0)
 		(effects
 			(font
@@
 	(symbol
 		(lib_id "Device:R_US")
-		(at 156.21 185.42 0)
+		(at 144.78 172.72 0)
 		(unit 1)
 		(exclude_from_sim no)
@@
 		(fields_autoplaced yes)
 		(property "Reference" "R11"
-			(at 158.75 184.1499 0)
+			(at 147.32 171.4499 0)
 			(effects
 				(font
@@
 		)
 		(property "Value" "R_US"
-			(at 158.75 186.6899 0)
+			(at 147.32 173.9899 0)
 			(effects
 				(font
@@
 		)
 		(property "Footprint" "Resistor_THT:R_Axial_DIN0207_L6.3mm_D2.5mm_P10.16mm_Horizontal"
-			(at 157.226 185.674 90)
+			(at 145.796 172.974 90)
 			(effects
 				(font
@@
 		)
 		(property "Datasheet" "~"
-			(at 156.21 185.42 0)
+			(at 144.78 172.72 0)
 			(effects
 				(font
@@
 		)
 		(property "Description" "Resistor, US symbol"
-			(at 156.21 185.42 0)
+			(at 144.78 172.72 0)
 			(effects
 				(font
@@
 	(symbol
 		(lib_id "Device:R_US")
-		(at 147.32 185.42 0)
+		(at 135.89 172.72 0)
 		(unit 1)
 		(exclude_from_sim no)
@@
 		(fields_autoplaced yes)
 		(property "Reference" "R10"
-			(at 149.86 184.1499 0)
+			(at 138.43 171.4499 0)
 			(effects
 				(font
@@
 		)
 		(property "Value" "R_US"
-			(at 149.86 186.6899 0)
+			(at 138.43 173.9899 0)
 			(effects
 				(font
@@
 		)
 		(property "Footprint" "Resistor_THT:R_Axial_DIN0207_L6.3mm_D2.5mm_P10.16mm_Horizontal"
-			(at 148.336 185.674 90)
+			(at 136.906 172.974 90)
 			(effects
 				(font
@@
 		)
 		(property "Datasheet" "~"
-			(at 147.32 185.42 0)
+			(at 135.89 172.72 0)
 			(effects
 				(font
@@
 		)
 		(property "Description" "Resistor, US symbol"
-			(at 147.32 185.42 0)
+			(at 135.89 172.72 0)
 			(effects
 				(font
@@
 	(symbol
 		(lib_id "Device:R_US")
-		(at 138.43 185.42 0)
+		(at 127 172.72 0)
 		(unit 1)
 		(exclude_from_sim no)
@@
 		(fields_autoplaced yes)
 		(property "Reference" "R9"
-			(at 140.97 184.1499 0)
+			(at 129.54 171.4499 0)
 			(effects
 				(font
@@
 		)
 		(property "Value" "R_US"
-			(at 140.97 186.6899 0)
+			(at 129.54 173.9899 0)
 			(effects
 				(font
@@
 		)
 		(property "Footprint" "Resistor_THT:R_Axial_DIN0207_L6.3mm_D2.5mm_P10.16mm_Horizontal"
-			(at 139.446 185.674 90)
+			(at 128.016 172.974 90)
 			(effects
 				(font
@@
 		)
 		(property "Datasheet" "~"
-			(at 138.43 185.42 0)
+			(at 127 172.72 0)
 			(effects
 				(font
@@
 		)
 		(property "Description" "Resistor, US symbol"
-			(at 138.43 185.42 0)
+			(at 127 172.72 0)
 			(effects
 				(font
@@
 	(symbol
 		(lib_id "LED:Inolux_IN-P55TATRGB")
-		(at 128.27 176.53 0)
+		(at 116.84 163.83 0)
 		(unit 1)
 		(exclude_from_sim no)
@@
 		(fields_autoplaced yes)
 		(property "Reference" "D3"
-			(at 128.27 166.37 0)
+			(at 116.84 153.67 0)
 			(effects
 				(font
@@
 		)
 		(property "Value" "Inolux_IN-P55TATRGB"
-			(at 128.27 168.91 0)
+			(at 116.84 156.21 0)
 			(effects
 				(font
@@
 		)
 		(property "Footprint" "LED_SMD:LED_Inolux_IN-P55TATRGB_PLCC6_5.0x5.5mm_P1.8mm"
-			(at 123.19 184.658 0)
+			(at 111.76 171.958 0)
 			(effects
 				(font
@@
 		)
 		(property "Datasheet" "https://www.inolux-corp.com/datasheet/SMDLED/RGB%20Top%20View/IN-P55TATRGB.pdf"
-			(at 123.19 186.69 0)
+			(at 111.76 173.99 0)
 			(effects
 				(font
@@
 		)
 		(property "Description" "Inolux RGB LED, PLCC-6"
-			(at 128.27 176.53 0)
+			(at 116.84 163.83 0)
 			(effects
 				(font
@@
 	(symbol
 		(lib_id "power:GND")
-		(at 147.32 189.23 0)
+		(at 135.89 176.53 0)
 		(unit 1)
 		(exclude_from_sim no)
@@
 		(fields_autoplaced yes)
 		(property "Reference" "#PWR07"
-			(at 147.32 195.58 0)
+			(at 135.89 182.88 0)
 			(effects
 				(font
@@
 		)
 		(property "Value" "GND"
-			(at 147.32 194.31 0)
+			(at 135.89 181.61 0)
 			(effects
 				(font
@@
 		)
 		(property "Footprint" ""
-			(at 147.32 189.23 0)
+			(at 135.89 176.53 0)
 			(effects
 				(font
@@
 		)
 		(property "Datasheet" ""
-			(at 147.32 189.23 0)
+			(at 135.89 176.53 0)
 			(effects
 				(font
@@
 		)
 		(property "Description" "Power symbol creates a global label with name \"GND\" , ground"
-			(at 147.32 189.23 0)
+			(at 135.89 176.53 0)
 			(effects
 				(font
@@
 	)
 	(symbol
-		(lib_id "Sensor_Optical:LDR07")
-		(at 177.8 115.57 0)
-		(unit 1)
-		(exclude_from_sim no)
-		(in_bom yes)
-		(on_board yes)
-		(dnp no)
-		(fields_autoplaced yes)
-		(property "Reference" "R1"
-			(at 180.34 114.2999 0)
-			(effects
-				(font
-					(size 1.27 1.27)
-				)
-				(justify left)
-			)
-		)
-		(property "Value" "LDR07"
-			(at 180.34 116.8399 0)
-			(effects
-				(font
-					(size 1.27 1.27)
-				)
-				(justify left)
-			)
-		)
-		(property "Footprint" "OptoDevice:R_LDR_5.1x4.3mm_P3.4mm_Vertical"
-			(at 182.245 115.57 90)
-			(effects
-				(font
-					(size 1.27 1.27)
-				)
-				(hide yes)
-			)
-		)
-		(property "Datasheet" "http://www.tme.eu/de/Document/f2e3ad76a925811312d226c31da4cd7e/LDR07.pdf"
-			(at 177.8 116.84 0)
-			(effects
-				(font
-					(size 1.27 1.27)
-				)
-				(hide yes)
-			)
-		)
-		(property "Description" "light dependent resistor"
-			(at 177.8 115.57 0)
-			(effects
-				(font
-					(size 1.27 1.27)
-				)
-				(hide yes)
-			)
-		)
-		(pin "2"
-		)
-		(pin "1"
-		)
-		(instances
-			(project ""
-				(path "/aa5a79bf-cc6f-4bf9-93a5-b1f0c6f58d36"
-					(reference "R1")
-					(unit 1)
-				)
-			)
-		)
-	)
-	(symbol
 		(lib_id "power:VCC")
 		(at 114.3 129.54 0)
@@
 					(unit 1)
 				)
-			)
-		)
-	)
-	(symbol
-		(lib_id "Switch:SW_Wuerth_450301014042")
-		(at 128.27 158.75 0)
-		(unit 1)
-		(exclude_from_sim no)
-		(in_bom yes)
-		(on_board yes)
-		(dnp no)
-		(fields_autoplaced yes)
-		(property "Reference" "SW1"
-			(at 128.27 149.86 0)
-			(effects
-				(font
-					(size 1.27 1.27)
-				)
-			)
-		)
-		(property "Value" "SW_Wuerth_450301014042"
-			(at 128.27 152.4 0)
-			(effects
-				(font
-					(size 1.27 1.27)
-				)
-			)
-		)
-		(property "Footprint" "Button_Switch_THT:SW_Slide-03_Wuerth-WS-SLTV_10x2.5x6.4_P2.54mm"
-			(at 128.27 168.91 0)
-			(effects
-				(font
-					(size 1.27 1.27)
-				)
-				(hide yes)
-			)
-		)
-		(property "Datasheet" "https://www.we-online.com/components/products/datasheet/450301014042.pdf"
-			(at 128.27 166.37 0)
-			(effects
-				(font
-					(size 1.27 1.27)
-				)
-				(hide yes)
-			)
-		)
-		(property "Description" "Switch slide, single pole double throw"
-			(at 128.27 158.75 0)
-			(effects
-				(font
-					(size 1.27 1.27)
-				)
-				(hide yes)
-			)
-		)
-		(pin "2"
-		)
-		(pin "1"
-		)
-		(pin "3"
-		)
-		(instances
-			(project ""
-				(path "/aa5a79bf-cc6f-4bf9-93a5-b1f0c6f58d36"
-					(reference "SW1")
-					(unit 1)
-				)
